Commit message: docs(hito1): añade reporte de definicion de juntas y validacion cruzada

File: Proyecto_Final/abb_irb120_urdf/urdf/abb_irb120.urdf (robot description, URDF)
Before this commit: robot abb_irb120, 8 links, 7 joints
Joints:
- joint joint_3: limit lower=-1.91986 upper=1.91986 effort=100 velocity=4.36332 -> lower=-1.91986 upper=1.22173 effort=100 velocity=4.36332

Commit message: fix(urdf): actualiza parametros del modelo abb irb 120 - limites modificados de los angulos de cada eslabon

File: Proyecto_Final/abb_irb120_urdf/urdf/abb_irb120.urdf (robot description, URDF)
Before this commit: robot abb_irb120, 8 links, 7 joints
Joints:
- joint joint_2: limit lower=-1.91986 upper=1.91986 effort=100 velocity=4.36332 -> lower=-1.22173 upper=1.22173 effort=100 velocity=4.36332
- joint joint_3: limit lower=-1.91986 upper=1.22173 effort=100 velocity=4.36332 -> lower=-1.74533 upper=0.78540 effort=100 velocity=4.36332
- joint joint_5: limit lower=-2.094395 upper=2.094395 effort=100 velocity=5.58505 -> lower=-1.57080 upper=1.57080 effort=100 velocity=5.58505
- joint joint_6: limit lower=-6.98132 upper=6.98132 effort=100 velocity=7.33038 -> lower=-3.14159 upper=3.14159 effort=100 velocity=7.33038
